File: RR_Lightdistance/RR_Lightdistance.kicad_sch (KiCad schematic)
At the start: 0 parts

Commit message: update schem
Changed lines of the file:
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@@
-	(wire
-		(pts
-			(xy 60.96 55.88) (xy 63.5 55.88)
-		)
-		(stroke
-			(width 0)
-			(type default)
-		)
-	)
 	(wire
 		(pts

Commit message: starting pcb
Other:
- sheet Laser ports: added none; removed GND_DIG
Changed lines of the file:
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@@
-	)
-	(junction
-		(at 71.12 100.33)
-		(diameter 0)
-		(color 0 0 0 0)
 	)
 	(junction
@@
 		(pts
 			(xy 138.43 63.5) (xy 138.43 83.82)
-		)
-		(stroke
-			(width 0)
-			(type default)
-		)
-	)
-	(wire
-		(pts
-			(xy 62.23 100.33) (xy 71.12 100.33)
 		)
 		(stroke
@@
 			)
 		)
-		(pin "GND_DIG" passive
-			(at 62.23 100.33 0)
-			(effects
-				(font
-					(size 1.27 1.27)
-				)
-				(justify right)
-			)
-		)

Commit message: mcp6004
Other:
- sheet Digital ports: added none; removed BOOST_EN
- sheet Laser ports: added 3V_DIG; removed 5V_LASER
- sheet Power ports: added none; removed 5V_LASER, BOOST_EN
Changed lines of the file:
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@@
+	)
+	(junction
+		(at 66.04 35.56)
+		(diameter 0)
+		(color 0 0 0 0)
 	)
 	(junction
@@
 	(wire
 		(pts
+			(xy 66.04 83.82) (xy 66.04 35.56)
+		)
+		(stroke
+			(width 0)
+			(type default)
+		)
+	)
+	(wire
+		(pts
 			(xy 82.55 110.49) (xy 113.03 110.49)
 		)
@@
 	(wire
 		(pts
-			(xy 46.99 80.01) (xy 46.99 64.77)
-		)
-		(stroke
-			(width 0)
-			(type default)
-		)
-	)
-	(wire
-		(pts
-			(xy 39.37 64.77) (xy 39.37 83.82)
-		)
-		(stroke
-			(width 0)
-			(type default)
-		)
-	)
-	(wire
-		(pts
 			(xy 101.6 129.54) (xy 101.6 30.48)
 		)
@@
 	(wire
 		(pts
-			(xy 60.96 35.56) (xy 99.06 35.56)
+			(xy 66.04 35.56) (xy 99.06 35.56)
+		)
+		(stroke
+			(width 0)
+			(type default)
+		)
+	)
+	(wire
+		(pts
+			(xy 60.96 35.56) (xy 66.04 35.56)
 		)
 		(stroke
@@
 	(wire
 		(pts
-			(xy 128.27 83.82) (xy 128.27 80.01)
-		)
-		(stroke
-			(width 0)
-			(type default)
-		)
-	)
-	(wire
-		(pts
 			(xy 60.96 30.48) (xy 101.6 30.48)
 		)
@@
 	(wire
 		(pts
+			(xy 55.88 83.82) (xy 66.04 83.82)
+		)
+		(stroke
+			(width 0)
+			(type default)
+		)
+	)
+	(wire
+		(pts
 			(xy 82.55 52.07) (xy 82.55 110.49)
 		)
@@
 		(pts
 			(xy 99.06 35.56) (xy 99.06 93.98)
-		)
-		(stroke
-			(width 0)
-			(type default)
-		)
-	)
-	(wire
-		(pts
-			(xy 46.99 80.01) (xy 128.27 80.01)
 		)
 		(stroke
@@
 			)
 		)
-		(pin "BOOST_EN" output
-			(at 128.27 83.82 90)
-			(effects
-				(font
-					(size 1.27 1.27)
-				)
-				(justify right)
-			)
-		)
 		(pin "3V3_ANA" input
 			(at 113.03 125.73 180)
@@
 			)
 		)
-		(pin "5V_LASER" output
-			(at 39.37 64.77 270)
-			(effects
-				(font
-					(size 1.27 1.27)
-				)
-				(justify left)
-			)
-		)
-		(pin "BOOST_EN" input
-			(at 46.99 64.77 270)
-			(effects
-				(font
-					(size 1.27 1.27)
-				)
-				(justify left)
-			)
-		)
 		(instances
 			(project "RR_Lightdistance"
@@
 			)
 		)
-		(pin "5V_LASER" input
-			(at 39.37 83.82 90)
-			(effects
-				(font
+		(pin "3V_DIG" input
+			(at 55.88 83.82 90)
+			(effects
+				(font
