File: RR_Lightdistance/digital.kicad_sch (KiCad schematic)
At the start: 7 parts, among them Q1 2N7002, U8 ESP32-C3_SUPERMINI_TH

Commit message: update schem
Connections:
- no-connect marks 0 -> 8
Changed lines of the file:
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@@
 		(color 0 0 0 0)
+	)
+	(no_connect
+		(at 111.76 57.15)
+	)
+	(no_connect
+		(at 76.2 46.99)
+	)
+	(no_connect
+		(at 111.76 52.07)
+	)
+	(no_connect
+		(at 111.76 44.45)
+	)
+	(no_connect
+		(at 111.76 54.61)
+	)
+	(no_connect
+		(at 76.2 49.53)
+	)
+	(no_connect
+		(at 76.2 57.15)
+	)
+	(no_connect
+		(at 76.2 59.69)
 	)
 	(wire

Commit message: starting pcb
Parts:
- C20, C21: footprint Package_SO:TSSOP-10_3x3mm_P0.5mm -> Capacitor_SMD:C_0603_1608Metric
- C22: footprint Package_SO:TSSOP-10_3x3mm_P0.5mm -> Capacitor_SMD:C_0805_2012Metric
- R14: footprint Package_TO_SOT_SMD:SOT-23 -> Resistor_SMD:R_0805_2012Metric
- analog2: footprint (none) -> Connector_JST:JST_PH_B4B-PH-K_1x04_P2.00mm_Vertical
Changed lines of the file:
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@@
 			)
 		)
-		(property "Footprint" "Package_SO:TSSOP-10_3x3mm_P0.5mm"
+		(property "Footprint" "Capacitor_SMD:C_0603_1608Metric"
 			(at 138.1252 46.99 0)
 			(hide yes)
@@
 			)
 		)
-		(property "Footprint" ""
+		(property "Footprint" "Connector_JST:JST_PH_B4B-PH-K_1x04_P2.00mm_Vertical"
 			(at 114.3 93.98 0)
 			(hide yes)
@@
 			)
 		)
-		(property "Footprint" "Package_TO_SOT_SMD:SOT-23"
+		(property "Footprint" "Resistor_SMD:R_0805_2012Metric"
 			(at 69.342 86.36 90)
 			(hide yes)
@@
 			)
 		)
-		(property "Footprint" "Package_SO:TSSOP-10_3x3mm_P0.5mm"
+		(property "Footprint" "Capacitor_SMD:C_0603_1608Metric"
 			(at 64.4652 59.69 0)
 			(hide yes)
@@
 			)
 		)
-		(property "Footprint" "Package_SO:TSSOP-10_3x3mm_P0.5mm"
+		(property "Footprint" "Capacitor_SMD:C_0805_2012Metric"
 			(at 130.5052 46.99 0)
 			(hide yes)

Commit message: firstpcb
Parts:
- removed C22: 10u, Capacitor_SMD:C_0805_2012Metric, symbol Device:C
- R14: footprint Resistor_SMD:R_0805_2012Metric -> Resistor_SMD:R_0603_1608Metric
- analog2: footprint Connector_JST:JST_PH_B4B-PH-K_1x04_P2.00mm_Vertical -> Connector_JST:JST_SH_BM04B-SRSS-TB_1x04-1MP_P1.00mm_Vertical
Connections:
- net BOOST_EN: now also U8.1 (GPIO1); no longer U8.3 (GPIO3)
- net SCL: now also U8.7 (GPIO7); no longer U8.9 (GPIO9)
- net VBAT_SENSE: now also U8.21 (GPIO21); no longer U8.0 (GPIO0)
- net at Q1.1 (G), R14.1: now also U8.0 (GPIO0); no longer U8.4 (GPIO4)

Commit message: mcp6004
Parts:
- removed C20: 100n, Capacitor_SMD:C_0603_1608Metric, symbol Device:C
Connections:
- net BOOST_EN: no longer names the net of U8.1 (GPIO1)
- no-connect marks 8 -> 9
Changed lines of the file:
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@@
-		(color 0 0 0 0)
-	)
-	(junction
-		(at 68.58 46.99)
-		(diameter 0)
 		(color 0 0 0 0)
 	)
@@
 	)
 	(no_connect
+		(at 76.2 46.99)
+	)
+	(no_connect
 		(at 76.2 57.15)
 	)
@@
 	(wire
 		(pts
-			(xy 68.58 46.99) (xy 76.2 46.99)
-		)
-		(stroke
-			(width 0)
-			(type default)
-		)
-	)
-	(wire
-		(pts
 			(xy 111.76 39.37) (xy 137.16 39.37)
 		)
@@
 		(pts
 			(xy 111.76 46.99) (xy 115.57 46.99)
-		)
-		(stroke
-			(width 0)
-			(type default)
-		)
-	)
-	(wire
-		(pts
-			(xy 68.58 46.99) (xy 62.23 46.99)
 		)
 		(stroke
@@
 		)
 	)
-	(hierarchical_label "BOOST_EN"
-		(shape output)
-		(at 62.23 46.99 180)
-		(effects
-			(font
-				(size 1.27 1.27)
-			)
-			(justify right)
-		)
-	)
 	(hierarchical_label "GND_DIG"
 		(shape passive)
@@
 		(shape input)
 		(at 109.22 96.52 180)
-		(effects
-			(font
-				(size 1.27 1.27)
-			)
-			(justify right)
-		)
-	)
-	(hierarchical_label "GND_DIG"
-		(shape passive)
-		(at 68.58 54.61 180)
 		(effects
 			(font
@@
 					(unit 1)
 				)
-			)
-		)
-	)
-	(symbol
-		(lib_id "Device:C")
-		(at 68.58 50.8 0)
-		(unit 1)
-		(body_style 1)
-		(exclude_from_sim no)
-		(in_bom yes)
-		(on_board yes)
-		(in_pos_files yes)
-		(dnp no)
-		(property "Reference" "C20"
-			(at 63.754 48.768 0)
-			(show_name no)
-			(do_not_autoplace no)
-			(effects
-				(font
-					(size 1.27 1.27)
-				)
-				(justify left)
-			)
-		)
-		(property "Value" "100n"
-			(at 63.246 52.832 0)
-			(show_name no)
-			(do_not_autoplace no)
-			(effects
-				(font
-					(size 1.27 1.27)
-				)
-				(justify left)
-			)
-		)
-		(property "Footprint" "Capacitor_SMD:C_0603_1608Metric"
-			(at 69.5452 54.61 0)
-			(hide yes)
-			(show_name no)
-			(do_not_autoplace no)
-			(effects
-				(font
-					(size 1.27 1.27)
-				)
-			)
-		)
-		(property "Datasheet" ""
-			(at 68.58 50.8 0)
-			(hide yes)
-			(show_name no)
-			(do_not_autoplace no)
-			(effects
-				(font
-					(size 1.27 1.27)
-				)
-			)
-		)
-		(property "Description" "Unpolarized capacitor"
-			(at 68.58 50.8 0)
-			(hide yes)
-			(show_name no)
-			(do_not_autoplace no)
-			(effects
-				(font
-					(size 1.27 1.27)
-				)
-			)
-		)
-		(pin "2"
-		)
-		(pin "1"
-		)
-		(instances
-			(project "RR_Lightdistance"
-				(path "/29467ab3-c1bf-4fb3-96d7-e47c1d2d2674/66b5f731-23bf-4488-a76d-6c2119f1b453"
-					(reference "C20")
-					(unit 1)
-				)
